Commit message: 官方camera、msg等配置更新

File: cyberdog_simulator/cyberdog_robot/cyberdog_description/xacro/robot.xacro (robot description, xacro)
@@ -2,5 +2,5 @@
 <robot name="cyber_dog" xmlns:xacro="http://www.ros.org/wiki/xacro">
     <xacro:arg name="ROBOT" default="cyber_dog" />
-    <xacro:arg name="USE_LIDAR" default="true" />
+    <xacro:arg name="USE_LIDAR" default="false" />
     <xacro:include filename="const.xacro" />
     <xacro:include filename="leg.xacro" />
@@ -77,5 +77,5 @@
         <parent link="body" />
         <child link="D435_camera_link" />
-        <origin rpy="0 0 0" xyz="271.994e-3 25e-3 114.912e-3" />
+        <origin rpy="0 1.0472 0" xyz="271.994e-3 25e-3 114.912e-3" />
     </joint>
     <link name="D435_camera_link">
